File: PCB/robot-boosterpack.kicad_pcb (KiCad board)
At the start: 2 copper layers, 60 x 90 mm, 59 parts, among them IC1 DRV8833, IC2 TPS77033, IC3 TPS77050, IC4 LMR61428, J1 3.3V Jumper, J2 5V Jumper, J3 9V Jumper, M1 MOTOR, M2 MOTOR

Commit message: fixed resistor placement for reflectance sensors
Parts:
- moved R11 2.00 mm to (200.0, 143.0)
- moved R8 2.00 mm to (200.0, 141.0)
- turned R1 to 180 degrees
- turned R13 to 180 degrees
- turned R15 to 180 degrees
- turned R6 to 180 degrees
- turned R7 to 180 degrees
Changed lines of the file:
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@@
   )
   (module SM0603 (layer B.Cu)
-    (at 200 143)
+    (at 200 141)
     (attr smd)
     (fp_text reference R8 (at 0 0) (layer B.SilkS)
@@
   )
   (module SM0603 (layer B.Cu)
-    (at 194 143)
-    (attr smd)
-    (fp_text reference R7 (at 0 0) (layer B.SilkS)
-      (effects (font (size 0.508 0.4572) (thickness 0.1143)) (justify mirror))
-    )
-    (fp_text value 10k (at 0 0) (layer B.SilkS) hide
-      (effects (font (size 0.508 0.4572) (thickness 0.1143)) (justify mirror))
-    )
-    (fp_line (start -1.143 0.635) (end 1.143 0.635) (layer B.SilkS) (width 0.127))
-    (fp_line (start 1.143 0.635) (end 1.143 -0.635) (layer B.SilkS) (width 0.127))
-    (fp_line (start 1.143 -0.635) (end -1.143 -0.635) (layer B.SilkS) (width 0.127))
-    (fp_line (start -1.143 -0.635) (end -1.143 0.635) (layer B.SilkS) (width 0.127))
-    (pad 1 smd rect (at -0.762 0) (size 0.635 1.143)
-      (layers B.Cu B.Paste B.Mask)
-      (net 1 +3.3V)
-    )
-    (pad 2 smd rect (at 0.762 0) (size 0.635 1.143)
+    (at 194 143 180)
+    (attr smd)
+    (fp_text reference R7 (at 0 0 180) (layer B.SilkS)
+      (effects (font (size 0.508 0.4572) (thickness 0.1143)) (justify mirror))
+    )
+    (fp_text value 10k (at 0 0 180) (layer B.SilkS) hide
+      (effects (font (size 0.508 0.4572) (thickness 0.1143)) (justify mirror))
+    )
+    (fp_line (start -1.143 0.635) (end 1.143 0.635) (layer B.SilkS) (width 0.127))
+    (fp_line (start 1.143 0.635) (end 1.143 -0.635) (layer B.SilkS) (width 0.127))
+    (fp_line (start 1.143 -0.635) (end -1.143 -0.635) (layer B.SilkS) (width 0.127))
+    (fp_line (start -1.143 -0.635) (end -1.143 0.635) (layer B.SilkS) (width 0.127))
+    (pad 1 smd rect (at -0.762 0 180) (size 0.635 1.143)
+      (layers B.Cu B.Paste B.Mask)
+      (net 1 +3.3V)
+    )
+    (pad 2 smd rect (at 0.762 0 180) (size 0.635 1.143)
       (layers B.Cu B.Paste B.Mask)
       (net 7 /IR2)
@@
   )
   (module SM0603 (layer B.Cu)
-    (at 200 141 180)
+    (at 200 143 180)
     (attr smd)
     (fp_text reference R11 (at 0 0 180) (layer B.SilkS)
@@
   )
   (module SM0603 (layer B.Cu)
-    (at 194 141)
-    (attr smd)
-    (fp_text reference R6 (at 0 0) (layer B.SilkS)
-      (effects (font (size 0.508 0.4572) (thickness 0.1143)) (justify mirror))
-    )
-    (fp_text value 100 (at 0 0) (layer B.SilkS) hide
-      (effects (font (size 0.508 0.4572) (thickness 0.1143)) (justify mirror))
-    )
-    (fp_line (start -1.143 0.635) (end 1.143 0.635) (layer B.SilkS) (width 0.127))
-    (fp_line (start 1.143 0.635) (end 1.143 -0.635) (layer B.SilkS) (width 0.127))
-    (fp_line (start 1.143 -0.635) (end -1.143 -0.635) (layer B.SilkS) (width 0.127))
-    (fp_line (start -1.143 -0.635) (end -1.143 0.635) (layer B.SilkS) (width 0.127))
-    (pad 1 smd rect (at -0.762 0) (size 0.635 1.143)
-      (layers B.Cu B.Paste B.Mask)
-      (net 1 +3.3V)
-    )
-    (pad 2 smd rect (at 0.762 0) (size 0.635 1.143)
+    (at 194 141 180)
+    (attr smd)
+    (fp_text reference R6 (at 0 0 180) (layer B.SilkS)
+      (effects (font (size 0.508 0.4572) (thickness 0.1143)) (justify mirror))
+    )
+    (fp_text value 100 (at 0 0 180) (layer B.SilkS) hide
+      (effects (font (size 0.508 0.4572) (thickness 0.1143)) (justify mirror))
+    )
+    (fp_line (start -1.143 0.635) (end 1.143 0.635) (layer B.SilkS) (width 0.127))
+    (fp_line (start 1.143 0.635) (end 1.143 -0.635) (layer B.SilkS) (width 0.127))
+    (fp_line (start 1.143 -0.635) (end -1.143 -0.635) (layer B.SilkS) (width 0.127))
+    (fp_line (start -1.143 -0.635) (end -1.143 0.635) (layer B.SilkS) (width 0.127))
+    (pad 1 smd rect (at -0.762 0 180) (size 0.635 1.143)
+      (layers B.Cu B.Paste B.Mask)
+      (net 1 +3.3V)
+    )
+    (pad 2 smd rect (at 0.762 0 180) (size 0.635 1.143)
       (layers B.Cu B.Paste B.Mask)
       (net 39 N-000008)
@@
   )
   (module SM0603 (layer B.Cu)
-    (at 206 143)
-    (attr smd)
-    (fp_text reference R13 (at 0 0) (layer B.SilkS)
-      (effects (font (size 0.508 0.4572) (thickness 0.1143)) (justify mirror))
-    )
-    (fp_text value 10k (at 0 0) (layer B.SilkS) hide
-      (effects (font (size 0.508 0.4572) (thickness 0.1143)) (justify mirror))
-    )
-    (fp_line (start -1.143 0.635) (end 1.143 0.635) (layer B.SilkS) (width 0.127))
-    (fp_line (start 1.143 0.635) (end 1.143 -0.635) (layer B.SilkS) (width 0.127))
-    (fp_line (start 1.143 -0.635) (end -1.143 -0.635) (layer B.SilkS) (width 0.127))
-    (fp_line (start -1.143 -0.635) (end -1.143 0.635) (layer B.SilkS) (width 0.127))
-    (pad 1 smd rect (at -0.762 0) (size 0.635 1.143)
-      (layers B.Cu B.Paste B.Mask)
-      (net 1 +3.3V)
-    )
-    (pad 2 smd rect (at 0.762 0) (size 0.635 1.143)
+    (at 206 143 180)
+    (attr smd)
+    (fp_text reference R13 (at 0 0 180) (layer B.SilkS)
+      (effects (font (size 0.508 0.4572) (thickness 0.1143)) (justify mirror))
+    )
+    (fp_text value 10k (at 0 0 180) (layer B.SilkS) hide
+      (effects (font (size 0.508 0.4572) (thickness 0.1143)) (justify mirror))
+    )
+    (fp_line (start -1.143 0.635) (end 1.143 0.635) (layer B.SilkS) (width 0.127))
+    (fp_line (start 1.143 0.635) (end 1.143 -0.635) (layer B.SilkS) (width 0.127))
+    (fp_line (start 1.143 -0.635) (end -1.143 -0.635) (layer B.SilkS) (width 0.127))
+    (fp_line (start -1.143 -0.635) (end -1.143 0.635) (layer B.SilkS) (width 0.127))
+    (pad 1 smd rect (at -0.762 0 180) (size 0.635 1.143)
+      (layers B.Cu B.Paste B.Mask)
+      (net 1 +3.3V)
+    )
+    (pad 2 smd rect (at 0.762 0 180) (size 0.635 1.143)
       (layers B.Cu B.Paste B.Mask)
       (net 9 /IR4)
@@
   )
   (module SM0603 (layer B.Cu)
-    (at 224 143)
-    (attr smd)
-    (fp_text reference R15 (at 0 0) (layer B.SilkS)
-      (effects (font (size 0.508 0.4572) (thickness 0.1143)) (justify mirror))
-    )
-    (fp_text value 10k (at 0 0) (layer B.SilkS) hide
-      (effects (font (size 0.508 0.4572) (thickness 0.1143)) (justify mirror))
-    )
-    (fp_line (start -1.143 0.635) (end 1.143 0.635) (layer B.SilkS) (width 0.127))
-    (fp_line (start 1.143 0.635) (end 1.143 -0.635) (layer B.SilkS) (width 0.127))
-    (fp_line (start 1.143 -0.635) (end -1.143 -0.635) (layer B.SilkS) (width 0.127))
-    (fp_line (start -1.143 -0.635) (end -1.143 0.635) (layer B.SilkS) (width 0.127))
-    (pad 1 smd rect (at -0.762 0) (size 0.635 1.143)
-      (layers B.Cu B.Paste B.Mask)
-      (net 1 +3.3V)
-    )
-    (pad 2 smd rect (at 0.762 0) (size 0.635 1.143)
+    (at 224 143 180)
+    (attr smd)
+    (fp_text reference R15 (at 0 0 180) (layer B.SilkS)
+      (effects (font (size 0.508 0.4572) (thickness 0.1143)) (justify mirror))
+    )
+    (fp_text value 10k (at 0 0 180) (layer B.SilkS) hide
+      (effects (font (size 0.508 0.4572) (thickness 0.1143)) (justify mirror))
+    )
+    (fp_line (start -1.143 0.635) (end 1.143 0.635) (layer B.SilkS) (width 0.127))
+    (fp_line (start 1.143 0.635) (end 1.143 -0.635) (layer B.SilkS) (width 0.127))
+    (fp_line (start 1.143 -0.635) (end -1.143 -0.635) (layer B.SilkS) (width 0.127))
+    (fp_line (start -1.143 -0.635) (end -1.143 0.635) (layer B.SilkS) (width 0.127))
+    (pad 1 smd rect (at -0.762 0 180) (size 0.635 1.143)
+      (layers B.Cu B.Paste B.Mask)
+      (net 1 +3.3V)
+    )
+    (pad 2 smd rect (at 0.762 0 180) (size 0.635 1.143)
       (layers B.Cu B.Paste B.Mask)
       (net 10 /IR5)
@@
   )
   (module SM0603 (layer B.Cu)
-    (at 176 141)
-    (attr smd)
-    (fp_text reference R1 (at 0 0) (layer B.SilkS)
-      (effects (font (size 0.508 0.4572) (thickness 0.1143)) (justify mirror))
-    )
-    (fp_text value 100 (at 0 0) (layer B.SilkS) hide
-      (effects (font (size 0.508 0.4572) (thickness 0.1143)) (justify mirror))
-    )
-    (fp_line (start -1.143 0.635) (end 1.143 0.635) (layer B.SilkS) (width 0.127))
-    (fp_line (start 1.143 0.635) (end 1.143 -0.635) (layer B.SilkS) (width 0.127))
-    (fp_line (start 1.143 -0.635) (end -1.143 -0.635) (layer B.SilkS) (width 0.127))
-    (fp_line (start -1.143 -0.635) (end -1.143 0.635) (layer B.SilkS) (width 0.127))
-    (pad 1 smd rect (at -0.762 0) (size 0.635 1.143)
-      (layers B.Cu B.Paste B.Mask)
-      (net 1 +3.3V)
-    )
-    (pad 2 smd rect (at 0.762 0) (size 0.635 1.143)
+    (at 176 141 180)
+    (attr smd)
+    (fp_text reference R1 (at 0 0 180) (layer B.SilkS)
+      (effects (font (size 0.508 0.4572) (thickness 0.1143)) (justify mirror))
+    )
+    (fp_text value 100 (at 0 0 180) (layer B.SilkS) hide
+      (effects (font (size 0.508 0.4572) (thickness 0.1143)) (justify mirror))
+    )
+    (fp_line (start -1.143 0.635) (end 1.143 0.635) (layer B.SilkS) (width 0.127))
+    (fp_line (start 1.143 0.635) (end 1.143 -0.635) (layer B.SilkS) (width 0.127))
+    (fp_line (start 1.143 -0.635) (end -1.143 -0.635) (layer B.SilkS) (width 0.127))
+    (fp_line (start -1.143 -0.635) (end -1.143 0.635) (layer B.SilkS) (width 0.127))
+    (pad 1 smd rect (at -0.762 0 180) (size 0.635 1.143)
+      (layers B.Cu B.Paste B.Mask)
+      (net 1 +3.3V)
+    )
+    (pad 2 smd rect (at 0.762 0 180) (size 0.635 1.143)
       (layers B.Cu B.Paste B.Mask)
       (net 20 N-0000016)
