File: PCB/robot-boosterpack.kicad_pcb (KiCad board)
At the start: 2 copper layers, 60 x 95 mm, 59 parts, among them IC1 DRV8833, IC2 TPS77033, IC3 TPS77050, IC4 LMR61428, J1 3.3V Jumper, J2 5V Jumper, J3 9V Jumper, M1 MOTOR, M2 MOTOR

Commit message: added battery drill module
Parts:
- added BATTERY: P***, 3xAAA, F.Cu at (200.0, 109.0)
- L1: moved to B.Cu
- moved M2 5.08 mm to (195.0, 84.0)
- moved C1 4.24 mm to (200.0, 68.8)
- moved C4 4.24 mm to (201.8, 70.5)
- moved C5 4.24 mm to (198.5, 70.5)
- moved IC1 4.24 mm to (201.0, 75.6)
- moved R5 4.24 mm to (202.3, 80.7)
- moved M1 4.04 mm to (205.0, 84.0), turned to 0 degrees
- turned L1 to 270 degrees
Changed lines of the file:
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@@
     (links 120)
     (no_connects 120)
-    (area 142.000002 59.539 254 156.217888)
+    (area 142.000002 50.150001 254 156.217888)
     (thickness 1.6)
     (drawings 16)
     (tracks 0)
     (zones 0)
-    (modules 59)
+    (modules 60)
     (nets 40)
   )
@@
   )
   (module tssop-16 (layer B.Cu)
-    (at 197.993 78.613 180)
+    (at 200.993 75.613 180)
     (descr TSSOP-16)
     (attr smd)
@@
   )
   (module SM0603_Capa (layer B.Cu)
-    (at 197 71.75 180)
+    (at 200 68.75 180)
     (attr smd)
     (fp_text reference C1 (at 0 0 450) (layer B.SilkS)
@@
   )
   (module SM0603_Capa (layer B.Cu)
-    (at 198.75 73.5 180)
+    (at 201.75 70.5 180)
     (attr smd)
     (fp_text reference C4 (at 0 0 450) (layer B.SilkS)
@@
   )
   (module SM0603_Capa (layer B.Cu)
-    (at 195.5 73.5)
+    (at 198.5 70.5)
     (attr smd)
     (fp_text reference C5 (at 0 0 270) (layer B.SilkS)
@@
   )
   (module SM0603 (layer B.Cu)
-    (at 199.263 83.693)
+    (at 202.263 80.693)
     (attr smd)
     (fp_text reference R5 (at 0 0) (layer B.SilkS)
@@
   )
   (module PIN_ARRAY_2X1 (layer F.Cu)
-    (at 208.28 86.36 180)
+    (at 205 84)
     (descr "Connecteurs 2 pins")
     (tags "CONN DEV")
-    (fp_text reference M1 (at 0 -1.905 180) (layer F.SilkS)
+    (fp_text reference M1 (at 0 -1.905) (layer F.SilkS)
       (effects (font (size 0.762 0.762) (thickness 0.1524)))
     )
-    (fp_text value MOTOR (at 0 -1.905 180) (layer F.SilkS) hide
+    (fp_text value MOTOR (at 0 -1.905) (layer F.SilkS) hide
       (effects (font (size 0.762 0.762) (thickness 0.1524)))
     )
@@
     (fp_line (start 2.54 -1.27) (end 2.54 1.27) (layer F.SilkS) (width 0.1524))
     (fp_line (start 2.54 1.27) (end -2.54 1.27) (layer F.SilkS) (width 0.1524))
-    (pad 1 thru_hole rect (at -1.27 0 180) (size 1.524 1.524) (drill 1.016)
+    (pad 1 thru_hole rect (at -1.27 0) (size 1.524 1.524) (drill 1.016)
       (layers *.Cu *.Mask F.SilkS)
       (net 37 N-0000059)
     )
-    (pad 2 thru_hole circle (at 1.27 0 180) (size 1.524 1.524) (drill 1.016)
+    (pad 2 thru_hole circle (at 1.27 0) (size 1.524 1.524) (drill 1.016)
       (layers *.Cu *.Mask F.SilkS)
       (net 36 N-0000058)
@@
   )
   (module PIN_ARRAY_2X1 (layer F.Cu)
-    (at 190.5 86.36)
+    (at 195 84)
     (descr "Connecteurs 2 pins")
     (tags "CONN DEV")
@@
     )
   )
-  (module INDUCTOR_SRN6045 (layer F.Cu)
-    (at 198.43 125.75 90)
-    (fp_text reference L1 (at 0 0 90) (layer F.SilkS)
-      (effects (font (size 1 1) (thickness 0.15)))
-    )
-    (fp_text value "6.8 uH" (at 0 0 90) (layer F.SilkS)
-      (effects (font (size 1 1) (thickness 0.15)))
-    )
-    (pad 1 smd rect (at -2.1 4 90) (size 2 6)
-      (layers F.Cu F.Paste F.Mask)
+  (module INDUCTOR_SRN6045 (layer B.Cu)
+    (at 198.43 125.75 270)
+    (fp_text reference L1 (at 0 0 270) (layer B.SilkS)
+      (effects (font (size 1 1) (thickness 0.15)) (justify mirror))
+    )
+    (fp_text value "6.8 uH" (at 0 0 270) (layer B.SilkS)
+      (effects (font (size 1 1) (thickness 0.15)) (justify mirror))
+    )
+    (pad 1 smd rect (at -2.1 -4 270) (size 2 6)
+      (layers B.Cu B.Paste B.Mask)
       (net 26 N-0000025)
     )
-    (pad 2 smd rect (at 2.2 4 90) (size 2 6)
-      (layers F.Cu F.Paste F.Mask)
+    (pad 2 smd rect (at 2.2 -4 270) (size 2 6)
+      (layers B.Cu B.Paste B.Mask)
       (net 23 N-0000020)
     )
@@
     )
   )
+  (module 3xAAA (layer F.Cu)
+    (at 200 109)
+    (descr "module 1 pin (ou trou mecanique de percage)")
+    (tags DEV)
+    (path 1pin)
+    (fp_text reference BATTERY (at 0 -5) (layer F.SilkS)
+      (effects (font (size 1.016 1.016) (thickness 0.254)))
+    )
+    (fp_text value P*** (at 0 2.794) (layer F.SilkS) hide
+      (effects (font (size 1.016 1.016) (thickness 0.254)))
+    )
+    (fp_line (start -18.415 25.6) (end 18.415 25.6) (layer F.SilkS) (width 0.15))
+    (fp_line (start 18.415 25.6) (end 18.415 -25.6) (layer F.SilkS) (width 0.15))
+    (fp_line (start 18.415 -25.6) (end -18.415 -25.6) (layer F.SilkS) (width 0.15))
+    (fp_line (start -18.415 -25.6) (end -18.415 25.6) (layer F.SilkS) (width 0.15))
+    (pad 1 thru_hole circle (at -14.605 0) (size 3 3) (drill 2.39)
+      (layers *.Cu *.Mask F.SilkS)
+    )
+    (pad 2 thru_hole circle (at 14.605 0) (size 3 3) (drill 2.39)
+      (layers *.Cu *.Mask F.SilkS)
+    )
+  )

Commit message: moved motor driver around to fit battery
Parts:
- moved R5 23.1 mm to (198.0, 58.0)
- moved M1 20.0 mm to (204.0, 64.0), turned to 180 degrees
- moved M2 20.0 mm to (195.0, 64.0), turned to 180 degrees
- moved C5 10.1 mm to (202.0, 80.0)
- moved C4 9.89 mm to (199.0, 80.0), turned to 0 degrees
- moved C1 9.25 mm to (200.0, 78.0)
- moved IC1 2.80 mm to (200.0, 73.0), turned to 0 degrees

Commit message: reoriented motor driver
Parts:
- moved C5 12.5 mm to (198.5, 68.0)
- moved C4 12.3 mm to (201.5, 68.0), turned to 180 degrees
- moved C1 12.0 mm to (200.0, 66.0)
- moved M1 3.00 mm to (207.0, 64.0)
- moved M2 2.00 mm to (193.0, 64.0)
- moved CONN2 1.41 mm to (200.0, 137.0)
- turned IC1 to 180 degrees
Changed lines of the file:
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@@
     (pad_to_mask_clearance 0)
     (aux_axis_origin 0 0)
-    (visible_elements 7FFFFBFF)
+    (visible_elements 7FFFFFFF)
     (pcbplotparams
       (layerselection 3178497)
@@
   )
   (module tssop-16 (layer B.Cu)
-    (at 200 73)
+    (at 200 73 180)
     (descr TSSOP-16)
     (attr smd)
-    (fp_text reference IC1 (at 0 -0.59944) (layer B.SilkS)
+    (fp_text reference IC1 (at 0 -0.59944 180) (layer B.SilkS)
       (effects (font (size 0.70104 0.59944) (thickness 0.11938)) (justify mirror))
     )
-    (fp_text value DRV8833 (at 0 1.00076) (layer B.SilkS)
+    (fp_text value DRV8833 (at 0 1.00076 180) (layer B.SilkS)
       (effects (font (size 1.00076 1.00076) (thickness 0.14986)) (justify mirror))
     )
@@
     (fp_line (start -2.54 -2.286) (end 2.54 -2.286) (layer B.SilkS) (width 0.127))
     (fp_line (start 2.54 -2.286) (end 2.54 2.286) (layer B.SilkS) (width 0.127))
-    (pad 4 smd rect (at -0.32512 -2.79908) (size 0.4191 1.47066)
+    (pad 4 smd rect (at -0.32512 -2.79908 180) (size 0.4191 1.47066)
       (layers B.Cu B.Paste B.Mask)
       (net 36 N-0000058)
     )
-    (pad 5 smd rect (at 0.32512 -2.79908) (size 0.4191 1.47066)
+    (pad 5 smd rect (at 0.32512 -2.79908 180) (size 0.4191 1.47066)
       (layers B.Cu B.Paste B.Mask)
       (net 35 N-0000057)
     )
-    (pad 6 smd rect (at 0.97536 -2.79908) (size 0.4191 1.47066)
-      (layers B.Cu B.Paste B.Mask)
-      (net 16 GND)
-    )
-    (pad 7 smd rect (at 1.6256 -2.79908) (size 0.4191 1.47066)
+    (pad 6 smd rect (at 0.97536 -2.79908 180) (size 0.4191 1.47066)
+      (layers B.Cu B.Paste B.Mask)
+      (net 16 GND)
+    )
+    (pad 7 smd rect (at 1.6256 -2.79908 180) (size 0.4191 1.47066)
       (layers B.Cu B.Paste B.Mask)
       (net 34 N-0000056)
     )
-    (pad 16 smd rect (at -2.26568 2.794) (size 0.4191 1.47066)
+    (pad 16 smd rect (at -2.26568 2.794 180) (size 0.4191 1.47066)
       (layers B.Cu B.Paste B.Mask)
       (net 11 /Left_Motor_1)
     )
-    (pad 1 smd rect (at -2.27584 -2.79908) (size 0.4191 1.47066)
+    (pad 1 smd rect (at -2.27584 -2.79908 180) (size 0.4191 1.47066)
       (layers B.Cu B.Paste B.Mask)
       (net 24 N-0000021)
     )
-    (pad 2 smd rect (at -1.6256 -2.79908) (size 0.4191 1.47066)
+    (pad 2 smd rect (at -1.6256 -2.79908 180) (size 0.4191 1.47066)
       (layers B.Cu B.Paste B.Mask)
       (net 37 N-0000059)
     )
-    (pad 3 smd rect (at -0.97536 -2.79908) (size 0.4191 1.47066)
-      (layers B.Cu B.Paste B.Mask)
-      (net 16 GND)
-    )
-    (pad 9 smd rect (at 2.27584 2.79908) (size 0.4191 1.47066)
+    (pad 3 smd rect (at -0.97536 -2.79908 180) (size 0.4191 1.47066)
+      (layers B.Cu B.Paste B.Mask)
+      (net 16 GND)
+    )
+    (pad 9 smd rect (at 2.27584 2.79908 180) (size 0.4191 1.47066)
       (layers B.Cu B.Paste B.Mask)
       (net 13 /Right_Motor_1)
     )
-    (pad 10 smd rect (at 1.6256 2.79908) (size 0.4191 1.47066)
+    (pad 10 smd rect (at 1.6256 2.79908 180) (size 0.4191 1.47066)
       (layers B.Cu B.Paste B.Mask)
       (net 14 /Right_Motor_2)
     )
-    (pad 11 smd rect (at 0.97536 2.79908) (size 0.4191 1.47066)
+    (pad 11 smd rect (at 0.97536 2.79908 180) (size 0.4191 1.47066)
       (layers B.Cu B.Paste B.Mask)
       (net 19 N-0000013)
     )
-    (pad 12 smd rect (at 0.32512 2.79908) (size 0.4191 1.47066)
+    (pad 12 smd rect (at 0.32512 2.79908 180) (size 0.4191 1.47066)
       (layers B.Cu B.Paste B.Mask)
       (net 3 +9V)
     )
-    (pad 13 smd rect (at -0.32512 2.79908) (size 0.4191 1.47066)
-      (layers B.Cu B.Paste B.Mask)
-      (net 16 GND)
-    )
-    (pad 14 smd rect (at -0.97536 2.79908) (size 0.4191 1.47066)
+    (pad 13 smd rect (at -0.32512 2.79908 180) (size 0.4191 1.47066)
+      (layers B.Cu B.Paste B.Mask)
+      (net 16 GND)
+    )
+    (pad 14 smd rect (at -0.97536 2.79908 180) (size 0.4191 1.47066)
       (layers B.Cu B.Paste B.Mask)
       (net 18 N-0000012)
     )
-    (pad 8 smd rect (at 2.27584 -2.79908) (size 0.4191 1.47066)
-      (layers B.Cu B.Paste B.Mask)
-    )
-    (pad 15 smd rect (at -1.6256 2.794) (size 0.4191 1.47066)
+    (pad 8 smd rect (at 2.27584 -2.79908 180) (size 0.4191 1.47066)
+      (layers B.Cu B.Paste B.Mask)
+    )
+    (pad 15 smd rect (at -1.6256 2.794 180) (size 0.4191 1.47066)
       (layers B.Cu B.Paste B.Mask)
       (net 12 /Left_Motor_2)
@@
   )
   (module SM0603_Capa (layer B.Cu)
-    (at 200 78 180)
+    (at 200 66 180)
     (attr smd)
     (fp_text reference C1 (at 0 0 450) (layer B.SilkS)
@@
   )
   (module SM0603_Capa (layer B.Cu)
-    (at 199 80)
-    (attr smd)
-    (fp_text reference C4 (at 0 0 270) (layer B.SilkS)
-      (effects (font (size 0.508 0.4572) (thickness 0.1143)) (justify mirror))
-    )
-    (fp_text value "2.2uF 6.3V" (at -1.651 0 270) (layer B.SilkS)
+    (at 201.5 68 180)
+    (attr smd)
+    (fp_text reference C4 (at 0 0 450) (layer B.SilkS)
+      (effects (font (size 0.508 0.4572) (thickness 0.1143)) (justify mirror))
+    )
+    (fp_text value "2.2uF 6.3V" (at -1.651 0 450) (layer B.SilkS)
+      (effects (font (size 0.508 0.4572) (thickness 0.1143)) (justify mirror))
+    )
+    (fp_line (start 0.50038 -0.65024) (end 1.19888 -0.65024) (layer B.SilkS) (width 0.11938))
+    (fp_line (start -0.50038 -0.65024) (end -1.19888 -0.65024) (layer B.SilkS) (width 0.11938))
+    (fp_line (start 0.50038 0.65024) (end 1.19888 0.65024) (layer B.SilkS) (width 0.11938))
+    (fp_line (start -1.19888 0.65024) (end -0.50038 0.65024) (layer B.SilkS) (width 0.11938))
+    (fp_line (start 1.19888 0.635) (end 1.19888 -0.635) (layer B.SilkS) (width 0.11938))
+    (fp_line (start -1.19888 -0.635) (end -1.19888 0.635) (layer B.SilkS) (width 0.11938))
+    (pad 1 smd rect (at -0.762 0 180) (size 0.635 1.143)
+      (layers B.Cu B.Paste B.Mask)
+      (net 18 N-0000012)
+    )
+    (pad 2 smd rect (at 0.762 0 180) (size 0.635 1.143)
+      (layers B.Cu B.Paste B.Mask)
+      (net 16 GND)
+    )
+    (model smd\capacitors\C0603.wrl
+      (at (xyz 0 0 0.001))
+      (scale (xyz 0.5 0.5 0.5))
+      (rotate (xyz 0 0 0))
+    )
+  )
+  (module SM0603_Capa (layer B.Cu)
+    (at 198.5 68)
+    (attr smd)
+    (fp_text reference C5 (at 0 0 270) (layer B.SilkS)
+      (effects (font (size 0.508 0.4572) (thickness 0.1143)) (justify mirror))
+    )
+    (fp_text value "0.01uF 16V X7R" (at -1.651 0 270) (layer B.SilkS)
       (effects (font (size 0.508 0.4572) (thickness 0.1143)) (justify mirror))
     )
@@
     (pad 1 smd rect (at -0.762 0) (size 0.635 1.143)
       (layers B.Cu B.Paste B.Mask)
-      (net 18 N-0000012)
+      (net 19 N-0000013)
     )
     (pad 2 smd rect (at 0.762 0) (size 0.635 1.143)
       (layers B.Cu B.Paste B.Mask)
-      (net 16 GND)
+      (net 3 +9V)
     )
     (model smd\capacitors\C0603.wrl
@@
   )
   (module SM0603_Capa (layer B.Cu)
-    (at 202 80)
-    (attr smd)
-    (fp_text reference C5 (at 0 0 270) (layer B.SilkS)
-      (effects (font (size 0.508 0.4572) (thickness 0.1143)) (justify mirror))
-    )
-    (fp_text value "0.01uF 16V X7R" (at -1.651 0 270) (layer B.SilkS)
+    (at 208.25 104.75)
+    (attr smd)
+    (fp_text reference C3 (at 0 0 270) (layer B.SilkS)
+      (effects (font (size 0.508 0.4572) (thickness 0.1143)) (justify mirror))
+    )
+    (fp_text value "1 uF" (at -1.651 0 270) (layer B.SilkS)
       (effects (font (size 0.508 0.4572) (thickness 0.1143)) (justify mirror))
     )
@@
     (pad 1 smd rect (at -0.762 0) (size 0.635 1.143)
       (layers B.Cu B.Paste B.Mask)
-      (net 19 N-0000013)
-    )
-    (pad 2 smd rect (at 0.762 0) (size 0.635 1.143)
-      (layers B.Cu B.Paste B.Mask)
-      (net 3 +9V)
-    )
-    (model smd\capacitors\C0603.wrl
-      (at (xyz 0 0 0.001))
-      (scale (xyz 0.5 0.5 0.5))
-      (rotate (xyz 0 0 0))
-    )
-  )
-  (module SM0603_Capa (layer B.Cu)
-    (at 208.25 104.75)
-    (attr smd)
-    (fp_text reference C3 (at 0 0 270) (layer B.SilkS)
-      (effects (font (size 0.508 0.4572) (thickness 0.1143)) (justify mirror))
-    )
-    (fp_text value "1 uF" (at -1.651 0 270) (layer B.SilkS)
-      (effects (font (size 0.508 0.4572) (thickness 0.1143)) (justify mirror))
-    )
-    (fp_line (start 0.50038 -0.65024) (end 1.19888 -0.65024) (layer B.SilkS) (width 0.11938))
-    (fp_line (start -0.50038 -0.65024) (end -1.19888 -0.65024) (layer B.SilkS) (width 0.11938))
-    (fp_line (start 0.50038 0.65024) (end 1.19888 0.65024) (layer B.SilkS) (width 0.11938))
-    (fp_line (start -1.19888 0.65024) (end -0.50038 0.65024) (layer B.SilkS) (width 0.11938))
-    (fp_line (start 1.19888 0.635) (end 1.19888 -0.635) (layer B.SilkS) (width 0.11938))
-    (fp_line (start -1.19888 -0.635) (end -1.19888 0.635) (layer B.SilkS) (width 0.11938))
-    (pad 1 smd rect (at -0.762 0) (size 0.635 1.143)
-      (layers B.Cu B.Paste B.Mask)
       (net 3 +9V)
     )
@@
   )
   (module PIN_ARRAY_2X1 (layer F.Cu)
-    (at 204 64 180)
+    (at 207 64 180)
     (descr "Connecteurs 2 pins")
     (tags "CONN DEV")
@@
   )
   (module PIN_ARRAY_2X1 (layer F.Cu)
-    (at 195 64 180)
+    (at 193 64 180)
     (descr "Connecteurs 2 pins")
     (tags "CONN DEV")
@@
   )
   (module PIN_ARRAY_2X1 (layer F.Cu)
-    (at 201 136 180)
+    (at 200 137 180)
     (descr "Connecteurs 2 pins")
     (tags "CONN DEV")

Commit message: replaced inductor with smaller part
Parts:
- L1: footprint INDUCTOR_SRN6045 -> NR6028T100M
- moved R5 20.2 mm to (200.5, 78.0)
- moved R22 6.34 mm to (205.5, 120.5), turned to 90 degrees
- moved L1 4.14 mm to (202.5, 126.5), turned to 180 degrees
- moved C8 2.28 mm to (196.0, 126.0)
- moved R19 1.00 mm to (196.0, 120.5)
- moved C9 0.99 mm to (194.0, 119.0)
- moved C11 0.98 mm to (207.0, 117.5), turned to 180 degrees
- moved C10 0.94 mm to (202.5, 117.5)
- moved R21 0.92 mm to (199.5, 117.5)
- moved R20 0.70 mm to (196.5, 118.0)
Changed lines of the file:
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@@
     (links 120)
     (no_connects 120)
-    (area 142.000002 50.150001 254 156.217888)
+    (area 142.000002 36.650001 254 168.7)
     (thickness 1.6)
-    (drawings 16)
+    (drawings 18)
     (tracks 0)
     (zones 0)
@@
       (drillshape 1)
       (scaleselection 1)
-      (outputdirectory ""))
+      (outputdirectory ../../../../Desktop/))
   )
   (net 0 "")
@@
   )
   (module SM1812 (layer B.Cu)
-    (at 193.731 126.227 90)
+    (at 196 126 90)
     (tags "CMS SM")
     (attr smd)
@@
   )
   (module SM1206POL (layer B.Cu)
-    (at 206.431 116.702 90)
-    (attr smd)
-    (fp_text reference C11 (at 0 0 90) (layer B.SilkS)
+    (at 207 117.5 180)
+    (attr smd)
+    (fp_text reference C11 (at 0 0 180) (layer B.SilkS)
       (effects (font (size 0.762 0.762) (thickness 0.127)) (justify mirror))
     )
-    (fp_text value 68uF (at 0 0 90) (layer B.SilkS) hide
+    (fp_text value 68uF (at 0 0 180) (layer B.SilkS) hide
       (effects (font (size 0.762 0.762) (thickness 0.127)) (justify mirror))
     )
@@
     (fp_line (start 2.54 -1.143) (end 0.889 -1.143) (layer B.SilkS) (width 0.127))
     (fp_line (start -0.889 1.143) (end -2.54 1.143) (layer B.SilkS) (width 0.127))
-    (pad 1 smd rect (at -1.651 0 90) (size 1.524 2.032)
+    (pad 1 smd rect (at -1.651 0 180) (size 1.524 2.032)
       (layers B.Cu B.Paste B.Mask)
       (net 3 +9V)
     )
-    (pad 2 smd rect (at 1.651 0 90) (size 1.524 2.032)
+    (pad 2 smd rect (at 1.651 0 180) (size 1.524 2.032)
       (layers B.Cu B.Paste B.Mask)
       (net 16 GND)
@@
   )
   (module SM0603_Capa (layer B.Cu)
-    (at 203.002 116.702)
+    (at 202.5 117.5)
     (attr smd)
     (fp_text reference C10 (at 0 0 270) (layer B.SilkS)
@@
   )
   (module SM0603_Capa (layer B.Cu)
-    (at 193.096 118.607 270)
+    (at 194 119 270)
     (attr smd)
     (fp_text reference C9 (at 0 0 540) (layer B.SilkS)
@@
   )
   (module SM0603 (layer B.Cu)
-    (at 203.002 114.67 180)
-    (attr smd)
-    (fp_text reference R22 (at 0 0 180) (layer B.SilkS)
-      (effects (font (size 0.508 0.4572) (thickness 0.1143)) (justify mirror))
-    )
-    (fp_text value 49.9 (at 0 0 180) (layer B.SilkS) hide
+    (at 205.5 120.5 90)
+    (attr smd)
+    (fp_text reference R22 (at 0 0 90) (layer B.SilkS)
+      (effects (font (size 0.508 0.4572) (thickness 0.1143)) (justify mirror))
+    )
+    (fp_text value 49.9 (at 0 0 90) (layer B.SilkS) hide
       (effects (font (size 0.508 0.4572) (thickness 0.1143)) (justify mirror))
     )
@@
     (fp_line (start 1.143 -0.635) (end -1.143 -0.635) (layer B.SilkS) (width 0.127))
     (fp_line (start -1.143 -0.635) (end -1.143 0.635) (layer B.SilkS) (width 0.127))
-    (pad 1 smd rect (at -0.762 0 180) (size 0.635 1.143)
+    (pad 1 smd rect (at -0.762 0 90) (size 0.635 1.143)
       (layers B.Cu B.Paste B.Mask)
       (net 26 N-0000025)
     )
-    (pad 2 smd rect (at 0.762 0 180) (size 0.635 1.143)
+    (pad 2 smd rect (at 0.762 0 90) (size 0.635 1.143)
       (layers B.Cu B.Paste B.Mask)
       (net 30 N-000003)
@@
   )
   (module SM0603 (layer B.Cu)
-    (at 196.271 117.337)
+    (at 196.5 118)
     (attr smd)
     (fp_text reference R20 (at 0 0) (layer B.SilkS)
@@
   )
   (module SM0603 (layer B.Cu)
-    (at 199.954 116.702 180)
+    (at 199.5 117.5 180)
     (attr smd)
     (fp_text reference R21 (at 0 0 180) (layer B.SilkS)
@@
   )
   (module SM0603 (layer B.Cu)
-    (at 195.001 120.512 90)
+    (at 196 120.5 90)
     (attr smd)
     (fp_text reference R19 (at 0 0 90) (layer B.SilkS)
@@
   )
   (module SM0603 (layer B.Cu)
-    (at 198 58)
+    (at 200.5 78)
     (attr smd)
     (fp_text reference R5 (at 0 0) (layer B.SilkS)
@@
     )
   )
-  (module INDUCTOR_SRN6045 (layer B.Cu)
-    (at 198.43 125.75 270)
-    (fp_text reference L1 (at 0 0 270) (layer B.SilkS)
-      (effects (font (size 1 1) (thickness 0.15)) (justify mirror))
-    )
-    (fp_text value "6.8 uH" (at 0 0 270) (layer B.SilkS)
-      (effects (font (size 1 1) (thickness 0.15)) (justify mirror))
-    )
-    (pad 1 smd rect (at -2.1 -4 270) (size 2 6)
-      (layers B.Cu B.Paste B.Mask)
-      (net 26 N-0000025)
-    )
-    (pad 2 smd rect (at 2.2 -4 270) (size 2 6)
-      (layers B.Cu B.Paste B.Mask)
-      (net 23 N-0000020)
-    )
-  )
   (module HEADER_2mm_1x3 (layer F.Cu)
     (at 200 146)
@@
     )
   )
+  (module NR6028T100M (layer B.Cu)
+    (at 202.5 126.5 180)
+    (fp_text reference L1 (at 0 5 180) (layer B.SilkS)
+      (effects (font (size 1 1) (thickness 0.15)) (justify mirror))
+    )
+    (fp_text value "6.8 uH" (at 0 -5 180) (layer B.SilkS)
+      (effects (font (size 1 1) (thickness 0.15)) (justify mirror))
+    )
+    (pad 1 smd rect (at -2.35 0 180) (size 1.6 5.7)
+      (layers B.Cu B.Paste B.Mask)
+      (net 26 N-0000025)
+    )
+    (pad 2 smd rect (at 2.35 0 180) (size 1.6 5.7)
+      (layers B.Cu B.Paste B.Mask)
+      (net 23 N-0000020)
+    )
+  )
+  (dimension 30 (width 0.3) (layer Cmts.User)
+    (gr_text "30.000 mm" (at 185.000001 38.150001) (layer Cmts.User)
+      (effects (font (size 1.5 1.5) (thickness 0.3)))
+    )
+    (feature1 (pts (xy 170 157) (xy 170.000001 36.800001)))
+    (feature2 (pts (xy 200 157) (xy 200.000001 36.800001)))
+    (crossbar (pts (xy 200.000001 39.500001) (xy 170.000001 39.500001)))
+    (arrow1a (pts (xy 170.000001 39.500001) (xy 171.126504 38.913581)))
+    (arrow1b (pts (xy 170.000001 39.500001) (xy 171.126504 40.086421)))
+    (arrow2a (pts (xy 200.000001 39.500001) (xy 198.873498 38.913581)))
+    (arrow2b (pts (xy 200.000001 39.500001) (xy 198.873498 40.086421)))
+  )
+  (dimension 60 (width 0.3) (layer Cmts.User)
+    (gr_text "60.000 mm" (at 200 167.349999) (layer Cmts.User)
+      (effects (font (size 1.5 1.5) (thickness 0.3)))
+    )
+    (feature1 (pts (xy 230 158) (xy 230 168.699999)))
+    (feature2 (pts (xy 170 158) (xy 170 168.699999)))
+    (crossbar (pts (xy 170 165.999999) (xy 230 165.999999)))
+    (arrow1a (pts (xy 230 165.999999) (xy 228.873497 166.586419)))
+    (arrow1b (pts (xy 230 165.999999) (xy 228.873497 165.413579)))
+    (arrow2a (pts (xy 170 165.999999) (xy 171.126503 166.586419)))
+    (arrow2b (pts (xy 170 165.999999) (xy 171.126503 165.413579)))
+  )
   (gr_line (start 229 67) (end 204 67) (angle 90) (layer Cmts.User) (width 0.2))
